File: pcb/kontakt.kicad_pcb (KiCad board)
At the start: 2 copper layers, 86 x 74 mm, 66 parts, among them CN1 Vin, CN2 5V, J1 UART, J2 LED_1, J3 LED2, J4 FAN1, J5 ARGB, J6 FAN2, J7 FAN3, J8 FAN4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

Commit message: Improved Kontakt PCB
Routing:
- net /rpi/QSPI_SCLK: track 11.0 -> 15.2 mm, vias 2 -> 0
- net /Peripherals/LED_2: track 47.3 -> 49.9 mm
- net GND: track 157.9 -> 159.4 mm, vias 145 -> 375
- net /rpi/QSPI_SS: track 18.2 -> 16.8 mm, vias 2 -> 0
- net /rpi/USB_D-: track 26.9 -> 25.8 mm
- net /Peripherals/FAN_3: track 47.8 -> 48.6 mm
- net /rpi/USB_D+: track 19.5 -> 20.3 mm
- net +1V1: track 31.6 -> 32.2 mm
- net /usb/D+: track 14.6 -> 14.0 mm
- net Net-(U1-USB_DM): track 15.5 -> 16.0 mm

Commit message: Improvements
Parts:
- removed G***: LOGO, LOGO
