File: pcb/peripherals.kicad_sch (KiCad schematic)
At the start: 14 parts, among them J1 UART, J2 LED_1, J3 LED2, J4 FAN1, J5 ARGB, J6 FAN2, J7 FAN3, J8 FAN4, Q1 IRLB8721PBF-VB, Q2 IRLB8721PBF-VB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

Commit message: Added case for pcb
Other:
- company: (none) -> playlogo
- title: (none) -> Kontakt
Changed lines of the file:
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@@
 	(generator_version "9.0")
 	(paper "A4")
+	(title_block
+		(title "Kontakt")
+		(date "2026-01-19")
+		(rev "2.0")
+		(company "playlogo")
+		(comment 4 "Peripherals")
+	)
 	(text "FANs"
 		(exclude_from_sim no)
