File: pcb/power.kicad_sch (KiCad schematic)
At the start: 10 parts, among them CN1 Vin, CN2 5V, U5 LM2596SX-5.0/NOPB, U6 CYA1050-47UH

Commit message: Added case for pcb
Other:
- company: (none) -> playlogo
- title: (none) -> Kontakt
Changed lines of the file:
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@@
 	(generator_version "9.0")
 	(paper "A4")
+	(title_block
+		(title "Kontakt")
+		(date "2026-01-19")
+		(rev "2.0")
+		(company "playlogo")
+		(comment 4 "PWR In & Step Down")
+	)
 	(text "24V Step down"
 		(exclude_from_sim no)
