File: pcb/rpi.kicad_sch (KiCad schematic)
At the start: 27 parts, among them SW1 GT-TC029A-H020-L1N, SW2 GT-TC029A-H020-L1N, U1 RP2040, U2 NCP1117ST33T3G, U3 W25Q128JVSIQ, U4 ABM8-272-T3_C20625731

Commit message: Added case for pcb
Other:
- company: (none) -> playlogo
- title: (none) -> Kontakt
Changed lines of the file:
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@@
 	(generator_version "9.0")
 	(paper "A4")
+	(title_block
+		(title "Kontakt")
+		(date "2026-01-19")
+		(rev "2.0")
+		(company "playlogo")
+		(comment 4 "RP2040 & supporting electronics")
+	)
 	(text "Flash"
 		(exclude_from_sim no)
