File: pcb/usb.kicad_sch (KiCad schematic)
At the start: 10 parts, among them U7 SL2.1A, U8 GT-USB-7010ASV

Commit message: Added case for pcb
Other:
- company: (none) -> playlogo
- title: (none) -> Kontakt
Changed lines of the file:
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@@
 	(generator_version "9.0")
 	(paper "A4")
+	(title_block
+		(title "Kontakt")
+		(date "2026-01-19")
+		(rev "2.0")
+		(company "playlogo")
+		(comment 4 "USB-C Input & Splitter")
+	)
 	(text "USB-C In"
 		(exclude_from_sim no)
